Commit message: Fix transformations

File: baxter_description/urdf/baxter_base/baxter_base.gazebo.xacro (robot description, xacro)
@@ -61,5 +61,5 @@
       <update_rate>30.0</update_rate>
       <camera name="head_camera">
-        <pose>0.0 0.21 0.0 0.0 -0.8 -1.570796327 </pose>
+        <pose>0 0 0 0 -1.57079632679 1.57079632679 </pose>
         <horizontal_fov>1.3962634</horizontal_fov>
         <image>

File: baxter_description/urdf/baxter_base/baxter_base.urdf.xacro (robot description, xacro)
@@ -231,5 +231,5 @@
     <!-- NICK PADILLA updated this to ensure the camera transformation is correct.-->
     <!-- <origin rpy="1.75057 0 1.57079632679" xyz="0.12839 0 0.06368"/> -->
-    <origin rpy="-2.53072 0 -1.57079632679" xyz="0.12839 0 0.06368"/>
+    <origin rpy="3.28318530718 0 -1.57079632679" xyz="0.22839 0 0.06368"/>
     <parent link="head"/>
     <child link="head_camera"/>
